Commit message: Added set_motor_for_joint for the front and back legs. Completed step 20

File: body.urdf (robot description, URDF)
Before this commit: robot robot, 3 links, 2 joints
Links:
- removed link Back_Leg
- removed link Front_Leg
- added link BackLeg, mass 1; collision box size=1 1 1; visual box size=1 1 1
- added link FrontLeg, mass 1; collision box size=1 1 1; visual box size=1 1 1
Joints:
- removed joint Torso_Back_Leg
- removed joint Torso_Front_Leg
- added joint Torso_BackLeg: type revolute, parent Torso, child BackLeg, origin xyz=-0.5 0 1 rpy=0 0 0, axis 0 1 0, limit lower=-3.14159 upper=3.14159 effort=0.0 velocity=0.0
- added joint Torso_FrontLeg: type revolute, parent Torso, child FrontLeg, origin xyz=0.5 0 1 rpy=0 0 0, axis 0 1 0, limit lower=-3.14159 upper=3.14159 effort=0.0 velocity=0.0
